Commit message: Update lerobot mash to match real robot. Now in pink ;)

File: ros_ws/src/lerobot/urdf/lerobot.urdf (robot description, URDF)
Before this commit: robot LeRobot, 8 links, 7 joints
Links:
- removed link Base
- removed link Fixed_Gripper
- removed link Lower_Arm
- removed link Moving_Jaw
- removed link Shoulder_Rotation_Pitch
- removed link Upper_Arm
- removed link Wrist_Pitch_Roll
- added link base, mass 1.0; collision mesh filename=package://lerobot/meshes/Base.stl; visual mesh filename=package://lerobot/meshes/Base.stl
- added link gripper, mass 0.0929859; visual mesh filename=package://lerobot/meshes/Fixed_Jaw.stl; visual mesh filename=package://lerobot/meshes/Fixed_Jaw_Motor.stl
- added link jaw, mass 0.0202444; visual mesh filename=package://lerobot/meshes/Moving_Jaw.stl
- added link lower_arm, mass 0.147968; collision mesh filename=package://lerobot/meshes/Lower_Arm.stl; visual mesh filename=package://lerobot/meshes/Lower_Arm.stl
- added link shoulder, mass 0.119226; collision mesh filename=package://lerobot/meshes/Rotation_Pitch.stl; visual mesh filename=package://lerobot/meshes/Rotation_Pitch.stl
- added link upper_arm, mass 0.162409; collision mesh filename=package://lerobot/meshes/Upper_Arm.stl; visual mesh filename=package://lerobot/meshes/Upper_Arm.stl
- added link wrist, mass 0.0661321; collision mesh filename=package://lerobot/meshes/Wrist_Pitch_Roll.stl; visual mesh filename=package://lerobot/meshes/Wrist_Pitch_Roll.stl
Joints:
- joint Elbow: axis 0 0 1 -> 1 0 0; child Lower_Arm -> lower_arm; limit lower=-1.57079632679 upper=1.57079632679 effort=10 velocity=10 -> lower=-3.14158 upper=0 effort=35 velocity=1; origin xyz=-0.11238 0.0282 0 rpy=0 0 -1.5708 -> xyz=0 0.11257 0.028 rpy=0 0 0; parent Upper_Arm -> upper_arm
- joint Gripper: child Moving_Jaw -> jaw; limit lower=0 upper=1.57079632679 effort=10 velocity=10 -> lower=-0.2 upper=2.0 effort=35 velocity=1; origin xyz=0.0202 0 0.024375 rpy=-1.5708 0 0 -> xyz=-0.0202 -0.0244 0 rpy=0 3.14158 0.15; parent Fixed_Gripper -> gripper
- joint Shoulder_Pitch: axis 0 0 1 -> 1 0 0; child Upper_Arm -> upper_arm; limit lower=-1.57079632679 upper=1.57079632679 effort=10 velocity=10 -> lower=0 upper=3.5 effort=35 velocity=1; origin xyz=0.000125 0.1086 0 rpy=3.1416 0 -1.5708 -> xyz=0 0.1025 0.0306 rpy=0.0 0 0; parent Shoulder_Rotation_Pitch -> shoulder
- joint Shoulder_Rotation: child Shoulder_Rotation_Pitch -> shoulder; limit lower=-1.57079632679 upper=1.57079632679 effort=10 velocity=10 -> lower=-2 upper=2 effort=35 velocity=1; origin xyz=0 -0.0452 0.0181 rpy=1.5708 0 1.5708 -> xyz=0 -0.0452 0.0165 rpy=1.57079 0 0; parent Base -> base
- joint Wrist_Pitch: child Wrist_Pitch_Roll -> wrist; limit lower=-1.57079632679 upper=1.57079632679 effort=10 velocity=10 -> lower=-2.5 upper=1.2 effort=35 velocity=1; origin xyz=-0.1102 0.005375 0 rpy=0 1.5708 0 -> xyz=0 0.0052 0.1349 rpy=-1.57079 0 0; parent Lower_Arm -> lower_arm
- joint Wrist_Roll: axis 0 0 1 -> 0 1 0; child Fixed_Gripper -> gripper; limit lower=-1.57079632679 upper=1.57079632679 effort=10 velocity=10 -> lower=-3.14158 upper=3.14158 effort=35 velocity=1; origin xyz=0 0.002 -0.0545 rpy=3.1416 0 3.1416 -> xyz=0 -0.0601 0 rpy=0 -1.57079 0; parent Wrist_Pitch_Roll -> wrist
- joint world_joint: child Base -> base

Commit message: Add a path publisher to edubot

File: ros_ws/src/lerobot/urdf/lerobot.urdf (robot description, URDF)
Before this commit: robot so_arm100, 8 links, 7 joints
Links:
- added link gripper_center
Joints:
- added joint Gripper_Center_Fixed: type fixed, parent gripper, child gripper_center, origin xyz=0.0 -0.075 0 rpy=0 0 0

Commit message: Change lerobot urdf to have all z-axes as rotaiton axes

File: ros_ws/src/lerobot/urdf/lerobot.urdf (robot description, URDF)
Before this commit: robot so_arm100, 9 links, 8 joints
Joints:
- joint Elbow: axis 1 0 0 -> 0 0 1; limit lower=-3.14158 upper=0 effort=35 velocity=1 -> lower=-1.58 upper=1.58 effort=35 velocity=1; origin xyz=0 0.11257 0.028 rpy=0 0 0 -> xyz=0.11257 -0.028 0 rpy=0 0 0
- joint Gripper: origin xyz=-0.0202 -0.0244 0 rpy=0 3.14158 0.15 -> xyz=-0.0202 0 0.0244 rpy=1.57079 3.14158 0.0
- joint Gripper_Center_Fixed: origin xyz=0.0 -0.075 0 rpy=0 0 0 -> xyz=0.0 0.0 0.075 rpy=0 0 0
- joint Shoulder_Pitch: axis 1 0 0 -> 0 0 1; limit lower=0 upper=3.5 effort=35 velocity=1 -> lower=-1.57 upper=1.57 effort=35 velocity=1; origin xyz=0 0.1025 0.0306 rpy=0.0 0 0 -> xyz=0 -0.0306 0.1025 rpy=0.0 -1.57079 0.0
- joint Shoulder_Rotation: axis 0 1 0 -> 0 0 1; origin xyz=0 -0.0452 0.0165 rpy=1.57079 0 0 -> xyz=0 -0.0452 0.0165 rpy=0 0 0
- joint Wrist_Pitch: axis 1 0 0 -> 0 0 1; limit lower=-2.5 upper=1.2 effort=35 velocity=1 -> lower=-1.57 upper=1.57 effort=35 velocity=1; origin xyz=0 0.0052 0.1349 rpy=-1.57079 0 0 -> xyz=0.0052 -0.1349 0 rpy=0 0 1.57079
- joint Wrist_Roll: axis 0 1 0 -> 0 0 1; origin xyz=0 -0.0601 0 rpy=0 -1.57079 0 -> xyz=-0.0601 0 0 rpy=0 -1.57079 0
- joint world_joint: origin xyz=0.0 0.0 0.0 rpy=0 0 0 -> xyz=0.0 0.0 0.0 rpy=0 0 3.14159

Commit message: Fix vis orientation of shoulder joing

File: ros_ws/src/lerobot/urdf/lerobot.urdf (robot description, URDF)
Before this commit: robot so_arm100, 9 links, 8 joints
Joints:
- joint Shoulder_Rotation: axis 0 0 1 -> 0 0 -1

Commit message: Properly fix direction of joint 0

File: ros_ws/src/lerobot/urdf/lerobot.urdf (robot description, URDF)
Before this commit: robot so_arm100, 9 links, 8 joints
Joints:
- joint Shoulder_Rotation: axis 0 0 -1 -> 0 0 1
